File: Robko01/Robko01.kicad_pcb (KiCad board)
At the start: 2 copper layers, 178.8 x 143.8 mm, 120 parts, among them J1 AC, J10 A_SEL, J11 Conn_01x02_Male, J2 BA, J3 BB, J4 AB, J5 BA, J6 AA, J7 MA, J8 MA, J9 MA, Q1 BD139, Q10 BD139, Q11 BD139, Q12 BD139, Q13 BD139, Q14 BD139, Q15 BD139, Q16 BD139, Q17 BD139, Q18 BD139, Q19 BD139, Q2 BD139, Q20 BD139, Q21 BD139, Q22 BD139, Q23 BD139, Q24 BD139, Q3 BD139, Q4 BD139, Q5 BD139, Q6 BD139, Q7 BD139, Q8 BD139, Q9 BD139, U1 7400, U10 74LS75, U11 74LS75, U12 7402, U13 7402, U14 7402, U15 7402, U16 7402, U17 74LS75, U18 74LS75, U19 74LS75, U2 74126, U20 74LS75, U21 74LS75, U22 74LS75, U23 7402, U24 7402, U25 7402, U3 74126, U4 7402, U5 L7805, U6 7407, U7 7407, U8 74LS04, U9 74LS138

Commit message: Update READEME
Other:
- board text added: "Orlin Dimitrov 2019 https://github.com/robko01/hw_main_board"
- board text removed: "Orlin Dimitrov 2019 http://github.com/orlin369/Robko01"
Changed lines of the file:
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@@
   )
   (page A4)
+  (title_block
+    (title "Rboko01 Main Board")
+    (rev 1.0)
+    (company 8BitClub)
+    (comment 1 "Orlin Dimitrov")
+    (comment 2 robko01@8bitclub.com)
+  )
   (layers
     (0 F.Cu signal)
@@
     )
   )
-  (gr_text "Orlin Dimitrov 2019\nhttp://github.com/orlin369/Robko01" (at 173.99 46.482 270) (layer F.Cu)
+  (gr_text "Orlin Dimitrov 2019\nhttps://github.com/robko01/hw_main_board" (at 173.99 46.482 270) (layer F.Cu)
     (effects (font (size 1.5 1.5) (thickness 0.375)))
   )
